File: whalepad-SI/whalepad.kicad_pcb (KiCad board)
At the start: 2 copper layers, 155.9 x 127.7 mm, 0 parts

Commit message: first proto rev
Parts:
- added C1: 4.7u, Capacitor_SMD:C_0402_1005Metric, F.Cu at (13.4, -27.0)
- added C10: 100n, Capacitor_SMD:C_0402_1005Metric, F.Cu at (46.1, -13.2)
- added C11: 100n, Capacitor_SMD:C_0402_1005Metric, F.Cu at (44.9, -13.2)
- added C12: 100n, Capacitor_SMD:C_0402_1005Metric, F.Cu at (6.08, -17.7)
- added C2: 1u, Capacitor_SMD:C_0402_1005Metric, F.Cu at (13.4, -25.8)
- added C3: 4.7u, Capacitor_SMD:C_0402_1005Metric, F.Cu at (25.2, -25.8)
- added C4: 1u, Capacitor_SMD:C_0402_1005Metric, F.Cu at (22.8, -25.8)
- added C5: 4.7u, Capacitor_SMD:C_0402_1005Metric, F.Cu at (16.2, -21.8)
- added C6: 1u, Capacitor_SMD:C_0402_1005Metric, F.Cu at (15.0, -21.8)
- added C7: 4.7u, Capacitor_SMD:C_0402_1005Metric, F.Cu at (8.19, -21.8)
- added C8: 1u, Capacitor_SMD:C_0402_1005Metric, F.Cu at (9.39, -21.8)
- added C9: 100n, Capacitor_SMD:C_0402_1005Metric, F.Cu at (21.7, -30.1)
- added D1: 1N4148WT, Diode_SMD:D_SOD-523, F.Cu at (14.3, -9.53)
- added D10: 1N4148WT, Diode_SMD:D_SOD-523, F.Cu at (23.8, 28.6)
- added D11: 1N4148WT, Diode_SMD:D_SOD-523, F.Cu at (33.3, 28.6)
- added D12: 1N4148WT, Diode_SMD:D_SOD-523, F.Cu at (14.3, 47.6)
- added D13: 1N4148WT, Diode_SMD:D_SOD-523, F.Cu at (23.8, 47.6)
- added D14: 1N4148WT, Diode_SMD:D_SOD-523, F.Cu at (33.3, 47.6)
- added D15: 1N4148WT, Diode_SMD:D_SOD-523, F.Cu at (42.9, 47.6)
- added D16: 1N4148WT, Diode_SMD:D_SOD-523, F.Cu at (33.3, 66.7)
- added D17: 1N4148WT, Diode_SMD:D_SOD-523, F.Cu at (42.9, 66.7)
- added D2: 1N4148WT, Diode_SMD:D_SOD-523, F.Cu at (23.8, -9.53)
- added D3: 1N4148WT, Diode_SMD:D_SOD-523, F.Cu at (33.3, -9.53)
- added D4: 1N4148WT, Diode_SMD:D_SOD-523, F.Cu at (42.9, -9.53)
- added D5: 1N4148WT, Diode_SMD:D_SOD-523, F.Cu at (14.3, 9.53)
- added D6: 1N4148WT, Diode_SMD:D_SOD-523, F.Cu at (23.8, 9.53)
- added D7: 1N4148WT, Diode_SMD:D_SOD-523, F.Cu at (33.3, 9.53)
- added D8: 1N4148WT, Diode_SMD:D_SOD-523, F.Cu at (42.9, 9.53)
- added D9: 1N4148WT, Diode_SMD:D_SOD-523, F.Cu at (14.3, 28.6)
- added F1: 500mA, Fuse:Fuse_0603_1608Metric, F.Cu at (24.0, -28.6)
- added F2: 500mA, Fuse:Fuse_0603_1608Metric, F.Cu at (8.02, -23.6)
- added G***: LOGO, logo-branding:SI, F.Cu at (-2.79, -26.5)
- added G***: LOGO, logo-branding:logo_silk_10, B.Cu at (-2.59, -26.3)
- added J1: USB_C_Receptacle_USB2.0, Connector_USB:USB_C_Receptacle_HRO_TYPE-C-31-M-12, F.Cu at (28.6, -37.7)
- added J2: BAT, Connector_Molex:Molex_PicoBlade_53048-0210_1x02_P1.25mm_Horizontal, B.Cu at (18.0, -12.2)
- added J3: Conn_01x07, Connector_Molex:Molex_PicoBlade_53048-0710_1x07_P1.25mm_Horizontal, B.Cu at (5.72, -12.2)
- added J4: JTAG_TC2030, marbastlib-various:CON_TC2030_outlined, B.Cu at (58.7, 11.0)
- added J5: RST, Connector_PinHeader_2.54mm:PinHeader_1x02_P2.54mm_Vertical, B.Cu at (64.6, -16.8)
- added L1: BLM15PX121SN1D, Inductor_SMD:L_0402_1005Metric, F.Cu at (24.0, -25.8)
- added L2: BLM15PX121SN1D, Inductor_SMD:L_0402_1005Metric, F.Cu at (21.7, -28.9)
- added Q1: AO3401A, Package_TO_SOT_SMD:SOT-23, F.Cu at (30.6, -12.7)
- added Q2: 2N7002, Package_TO_SOT_SMD:SOT-23, F.Cu at (36.1, -12.7)
- added R1: 5k1, Resistor_SMD:R_0402_1005Metric, F.Cu at (17.3, -31.3)
- added R10: 5k1, Resistor_SMD:R_0402_1005Metric, F.Cu at (46.1, -15.4)
- added R11: 10k, Resistor_SMD:R_0402_1005Metric, F.Cu at (33.4, -13.7)
- added R12: 100R, Resistor_SMD:R_0402_1005Metric, F.Cu at (46.1, -19.6)
- added R13: 10k, Resistor_SMD:R_0402_1005Metric, F.Cu at (44.9, -19.6)
- added R2: 5k1, Resistor_SMD:R_0402_1005Metric, F.Cu at (14.6, -31.3)
- added R3: 10k, Resistor_SMD:R_0402_1005Metric, F.Cu at (8.99, -25.0)
- added R4: 22k, Resistor_SMD:R_0402_1005Metric, F.Cu at (11.0, -27.0)
- added R5: 2k2, Resistor_SMD:R_0402_1005Metric, F.Cu at (15.0, -24.2)
- added R6: 2k2, Resistor_SMD:R_0402_1005Metric, F.Cu at (11.0, -25.8)
- added R7: 10k, Resistor_SMD:R_0402_1005Metric, F.Cu at (13.7, -19.7)
- added R8: 1M, Resistor_SMD:R_0402_1005Metric, F.Cu at (21.7, -31.3)
- added R9: 5k1, Resistor_SMD:R_0402_1005Metric, F.Cu at (44.9, -15.4)
- added S1: MX_stab, marbastlib-mx:STAB_MX_P_2u, F.Cu at (57.1, 28.6)
- added S2: MX_stab, marbastlib-mx:STAB_MX_P_2u, F.Cu at (57.1, 66.7)
- added S3: MX_stab, marbastlib-mx:STAB_MX_P_2u, F.Cu at (9.53, 76.2)
- added SW1: SW, marbastlib-hitek:SW_HiTek_MX_1u, F.Cu at (0.00, 0.00)
- added SW10: SW, marbastlib-hitek:SW_HiTek_MX_1u, F.Cu at (19.1, 38.1)
- added SW11: SW, marbastlib-hitek:SW_HiTek_MX_1u, F.Cu at (38.1, 38.1)
- added SW12: SW, marbastlib-hitek:SW_HiTek_MX_1u, F.Cu at (0.00, 57.1)
- added SW13: SW, marbastlib-hitek:SW_HiTek_MX_1u, F.Cu at (19.1, 57.1)
- added SW14: SW, marbastlib-hitek:SW_HiTek_MX_1u, F.Cu at (38.1, 57.1)
- added SW15: SW, marbastlib-hitek:SW_HiTek_MX_1u, F.Cu at (57.1, 66.7)
- added SW16: SW, marbastlib-hitek:SW_HiTek_MX_1u, F.Cu at (9.53, 76.2)
- added SW17: SW, marbastlib-hitek:SW_HiTek_MX_1u, F.Cu at (38.1, 76.2)
- added SW2: SW, marbastlib-hitek:SW_HiTek_MX_1u, F.Cu at (19.1, 0.00)
- added SW3: SW, marbastlib-hitek:SW_HiTek_MX_1u, F.Cu at (38.1, 0.00)
- added SW4: SW, marbastlib-hitek:SW_HiTek_MX_1u, F.Cu at (57.1, 0.00)
- added SW5: SW, marbastlib-hitek:SW_HiTek_MX_1u, F.Cu at (0.00, 19.1)
- added SW6: SW, marbastlib-hitek:SW_HiTek_MX_1u, F.Cu at (19.1, 19.1)
- added SW7: SW, marbastlib-hitek:SW_HiTek_MX_1u, F.Cu at (38.1, 19.1)
- added SW8: SW, marbastlib-hitek:SW_HiTek_MX_1u, F.Cu at (57.1, 28.6)
- added SW9: SW, marbastlib-hitek:SW_HiTek_MX_1u, F.Cu at (0.00, 38.1)
- added U1: SRV05-4, Package_TO_SOT_SMD:SOT-23-6, F.Cu at (28.1, -23.7)
- added U2: BQ24075RGT, Package_DFN_QFN:VQFN-16-1EP_3x3mm_P0.5mm_EP1.6x1.6mm, F.Cu at (12.2, -23.0)
- added U3: MAX17048, Package_DFN_QFN:DFN-8-1EP_2x2mm_P0.5mm_EP0.7x1.3mm, F.Cu at (8.28, -17.2)
- added U4: nRF52840_moko_mk08, marbastlib-various:nRF52840_moko_mk08, F.Cu at (54.8, -19.0)
Routing:
- net c0: track 0.00 -> 152.5 mm
- net c1: track 0.00 -> 110.5 mm
- net c2: track 0.00 -> 107.7 mm
- net r4: track 0.00 -> 105.1 mm
- net r3: track 0.00 -> 100.5 mm
- net c3: track 0.00 -> 90.0 mm
- net VDDH: track 0.00 -> 87.4 mm, vias 0 -> 4
- net r2: track 0.00 -> 76.5 mm
- net +5V: track 0.00 -> 75.9 mm, vias 0 -> 2
- net USB_D+: track 0.00 -> 69.8 mm, vias 0 -> 1
- net USB_D-: track 0.00 -> 67.5 mm, vias 0 -> 1
- net SDA: track 0.00 -> 54.1 mm, vias 0 -> 1
- net SCL: track 0.00 -> 52.4 mm, vias 0 -> 1
- net r1: track 0.00 -> 52.3 mm
- net VDD: track 0.00 -> 51.2 mm, vias 0 -> 3
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- added copper zone on F.Cu, net Earth
- added copper zone on B.Cu, net GND
- added copper zone on F.Cu, net GND
Other:
- board size 155.9 x 127.7 mm -> 76.2 x 127.3 mm
- board text added: "1.09"
- board text added: "BAT+"
- board text added: "BAT-"
- board text added: "GND"
- board text added: "J2"
- board text added: "JLCJLCJLCJLC"
- board text added: "P1.09"
- board text added: "RST"
- board text added: "SCL"
- board text added: "SDA"
- board text added: "SWD"
- board text added: "VDDH"
- board text added: "VSW"
- board text added: "github.com/ebastler/wlpad mpwr.xyz rc1.0"
- board text added: "~{CHG}"
