File: plate-SI/plate-SI.kicad_pcb (KiCad board)
At the start: 2 copper layers, 77.2 x 127.7 mm, 10 parts, among them J1 Conn_01x07, J2 Conn_01x04

Commit message: fixed SI plate, added MX plate
Parts:
- J1: value Conn_01x07 -> EXT
- J2: value Conn_01x04 -> OLED
- LED1: renamed from D1; footprint marbastlib-various:LED_WS2812_2020 -> PCM_marbastlib-various:LED_WS2812_2020
- LED2: renamed from D2; footprint marbastlib-various:LED_WS2812_2020 -> PCM_marbastlib-various:LED_WS2812_2020
- LED3: renamed from D3; footprint marbastlib-various:LED_WS2812_2020 -> PCM_marbastlib-various:LED_WS2812_2020
- LED4: renamed from D4; footprint marbastlib-various:LED_WS2812_2020 -> PCM_marbastlib-various:LED_WS2812_2020
- LED5: renamed from D5; footprint marbastlib-various:LED_WS2812_2020 -> PCM_marbastlib-various:LED_WS2812_2020
- LED6: renamed from D6; footprint marbastlib-various:LED_WS2812_2020 -> PCM_marbastlib-various:LED_WS2812_2020
- renumbered D7 to D1, D8 to D2
Connections:
- D1 pad 1: GND -> LED_CHG
- D1 pad 2: LED_CHG -> VDDH
- D2 pad 1: GND -> LED_CHG
- D2 pad 2: LED_CHG -> VDDH
Routing:
- net GND: track 132.5 -> 49.1 mm
- net VDDH: track 0.00 -> 79.3 mm
- net LED_CHG: track 80.3 -> 78.7 mm
Other:
- outline, holes or cut-outs redrawn
